File: schematics/xray/xray.kicad_pcb (KiCad board)
At the start: 4 copper layers, 130 x 65 mm, 118 parts, among them J1 USB_A, J2 USB_B_Micro, J3 USB_C_Receptacle_USB2.0, J4 USBASP, M1 VibroMotor, 3V, 8x2.7mm, Q1 IRF7413ZPbF, Q10 IRLML5203, Q11 IRLML0030, Q12 IRLML0030, Q13 IRLML0030, Q14 IRLML0030, Q2 IRF7424PBF, Q3 IRLML0030, Q4 IRF7424PBF, Q5 BC857, Q6 IRLML0030, Q7 BC847, Q8 IRLML0030, Q9 IRLML5203, SW1 EC11W****, SW2 B3F3150, T1 Transformer_1P_1S, U1 PCA9306, U2 IP5328P, U3 ATmega328P-A, U4 SN74LVC2T45DCUR, U5 SN74LVC2T45DCUR, U6 SN74LVC2T45DCUR, U7 Display_1.18inch_st7535, Y1 HC-49SM, 8MHz

Commit message: board production started
Parts:
- removed the L1 at (150.0, 89.5)
- removed the R32 at (101.1, 126.0)
- added H1: MountingHole, MountingHole:MountingHole_3.2mm_M3, F.Cu at (132.2, 97.8)
- added H3: MountingHole, MountingHole:MountingHole_3.2mm_M3, F.Cu at (113.0, 120.8)
- added JP1: SolderJumper_2_Open, Jumper:SolderJumper-2_P1.3mm_Open_TrianglePad1.0x1.5mm, B.Cu at (91.0, 85.0)
- added R26: 0, Resistor_SMD:R_1206_3216Metric, F.Cu at (86.9, 112.6)
- added R28: 0, Resistor_SMD:R_1206_3216Metric, F.Cu at (108.3, 115.2)
- added R29: 0, Resistor_SMD:R_1206_3216Metric, F.Cu at (86.9, 116.6)
- C11, C8, C9: value 0.1 uF, 630V -> К73-17, 0.1 uF, 630V
- C12, C38, Q12, R14: moved to B.Cu
- C18, C19, Q13, R1: moved to F.Cu
- C22: renamed from C23; moved to B.Cu
- C23: renamed from C24; value 100 nF -> 470 nF
- C24: renamed from C20; value ~10 pF, 630V -> CC81, 10 pF, 630V
- C30, C31, C5, C7: footprint Capacitor_SMD:C_1206_3216Metric -> Capacitor_SMD:C_0603_1608Metric
- C32: renamed from C33; footprint Capacitor_SMD:C_1206_3216Metric -> Capacitor_SMD:C_0603_1608Metric; moved to B.Cu
- C33: renamed from C34; footprint Capacitor_SMD:C_1206_3216Metric -> Capacitor_SMD:C_0603_1608Metric
- C34: renamed from C32; footprint Capacitor_SMD:C_1206_3216Metric -> Capacitor_SMD:C_0603_1608Metric
- C6: value see note LC* -> see note [*]; footprint Capacitor_SMD:C_1206_3216Metric -> Capacitor_SMD:C_0603_1608Metric
- D3: footprint Diode_SMD:D_SMA -> Diode_THT:D_5W_P5.08mm_Vertical_AnodeUp; moved to F.Cu
- F1: value 1808, 6.3A -> 1808, 6A
- L2: renamed from L3; value 10 uH -> 20 uH; footprint Capacitor_SMD:C_1210_3225Metric -> Inductor_SMD:L_1210_3225Metric
- Q1: value IRF7413ZPbF -> IRF7832PbF
- Q2, Q4: value IRF7424PBF -> IRF7425PbF; footprint Package_SO:SO-8_3.9x4.9mm_P1.27mm -> Package_SO:SOIC-8_3.9x4.9mm_P1.27mm
- R16: renamed from R17; footprint Resistor_SMD:R_0805_2012Metric -> Resistor_SMD:R_1206_3216Metric
- R17: renamed from R15; value 200K** (82K ?) -> 67K**
- R24: renamed from R25; value RSET [?] -> VSET [?]; moved to F.Cu
- R31: renamed from R28; value 200K -> 400K
- R33: renamed from R30; value 0 ? -> 0; footprint Resistor_SMD:R_0805_2012Metric -> Resistor_SMD:R_1206_3216Metric
- R34: renamed from R31; moved to B.Cu
- R35: renamed from R33; moved to F.Cu
- moved C38 49.2 mm to (98.8, 135.6), turned to 0 degrees
- moved R7 35.0 mm to (153.8, 83.5), turned to 0 degrees
- moved C32 33.4 mm to (165.5, 82.2), turned to -90 degrees
- moved C7 32.5 mm to (156.3, 86.3), turned to 180 degrees
- moved U1 27.7 mm to (156.3, 89.8), turned to 180 degrees
- moved C22 23.6 mm to (152.5, 101.3), turned to 180 degrees
- moved C33 16.9 mm to (176.0, 112.5), turned to -90 degrees
- moved C19 16.0 mm to (160.3, 107.8)
- moved C10 13.4 mm to (163.0, 93.8), turned to 180 degrees
- moved C20 10.8 mm to (152.5, 101.3), turned to 180 degrees
- moved R24 9.89 mm to (149.3, 134.0)
- moved Q6 8.25 mm to (161.3, 134.3)
- moved C21 8.04 mm to (152.5, 97.3), turned to 180 degrees
- moved R18 7.99 mm to (161.3, 130.5)
- moved R22 7.50 mm to (161.3, 137.5)
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- renumbered C21 to C20, C22 to C21, J2 to J1, J1 to J2, JP1 to JP2, L2 to L1, R8 to R10, R9 to R11, R16 to R15, R20 to R18, R21 to R19, R22 to R20, R18 to R21, R23 to R22, R19 to R23, R24 to R25, R26 to R27, R27 to R30, R29 to R32, R10 to R8, R11 to R9
Connections:
- net DCDC_L renamed Net-(C18-Pad2)
- D4 pad 2: VCC -> Net-(D4-Pad2)
- D5 pad 2: VCC -> Net-(D5-Pad2)
- D6 pad 2: VCC -> Net-(D6-Pad2)
- R1 pad 1: Net-(L1-Pad2) -> VCC
- R10 pad 1: Net-(C11-Pad2) -> Net-(JP1-Pad2)
- R31 pad 1: Net-(R28-Pad1) -> Net-(C40-Pad1)
Routing:
- net VCC: track 387.5 -> 184.8 mm, vias 12 -> 8
- net GND: track 632.8 -> 530.4 mm, vias 11 -> 12
- net VREG: track 89.0 -> 54.1 mm, vias 4 -> 2
- net Net-(D4-Pad2): track 0.00 -> 31.6 mm
- net Net-(D6-Pad2): track 0.00 -> 27.8 mm
- net USB_VMID: track 123.8 -> 96.1 mm
- net TXD: track 59.9 -> 34.6 mm
- net MCU_I2C_SDA: track 6.42 -> 31.3 mm, vias 1 -> 2
- net MCU_I2C_SCL: track 9.22 -> 32.0 mm, vias 1 -> 2
- net USB_I2C_SDA: track 44.5 -> 25.4 mm, vias 2 -> 1
- net USB_I2C_SCL: track 44.6 -> 25.6 mm, vias 2 -> 1
- net FLASHLIGHT: track 59.1 -> 41.4 mm, vias 2 -> 1
- net USB_INT: track 36.5 -> 49.4 mm
- net unconnected-(J2-Pad5): track 26.3 -> 14.5 mm
- net Net-(C7-Pad2): track 17.4 -> 6.68 mm
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- removed copper zone on F.Cu, net GND
- removed copper zone on In2.Cu, net GND
- removed copper zone on F.Cu, net Net-(C18-Pad2)
- removed copper zone on F.Cu, net USB_IN_VBUS
- removed copper zone on F.Cu, net USB_M_IN_VBUS
- removed copper zone on F.Cu, net USB_OUT_VBUS
- removed copper zone on F.Cu, net USB_VMID
- removed copper zone on In1.Cu, net USB_VMID
- removed copper zone on F.Cu, net USB_VSYS
- removed copper zone on In2.Cu, net VCC
Other:
- board text added: "D3 place"

Commit message: Intermediate commit before re-writing ATMega and IP5328 integration
Parts:
- R26, R29: value 0 -> 16
- R28: value 0 -> 27
- R9: value 100K@25C -> NTCM-100K@25-B4250

Commit message: Prepare to re-write UI
Parts:
- C34: value 200 pF*** -> 330 pF***
- R24: value VSET [?] -> 510K
- R31: value 400K -> 400K ****
- R33: value 0 -> 27
Changed lines of the file:
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@@
   (net 15 "USB_OUT_D-")
   (net 16 "USB_OUT_D+")
-  (net 17 "Net-(#FLG03-pwr)")
+  (net 17 "Net-(U1-EN)")
   (net 18 "USB_IN_CC1")
   (net 19 "+5V")
@@
   (net 47 "MISO")
   (net 48 "SCK")
-  (net 49 "Net-(#FLG04-pwr)")
+  (net 49 "Net-(U3-AVCC)")
   (net 50 "Net-(Q5-B)")
   (net 51 "Net-(R11-Pad2)")
@@
   (net 88 "Net-(Q6-D)")
   (net 89 "Net-(Q9-D)")
-  (net 90 "Net-(#FLG08-pwr)")
+  (net 90 "Net-(Q10-D)")
   (net 91 "Net-(U2-RSET)")
   (net 92 "unconnected-(U2-DPA2-Pad1)")
@@
       (stroke (width 0.1) (type solid)) (layer "F.Fab"))
     (pad "1" smd roundrect (at -0.775 0) (size 0.9 0.95) (layers "F.Cu" "F.Paste" "F.Mask") (roundrect_rratio 0.25)
-      (net 49 "Net-(#FLG04-pwr)") (pintype "passive"))
+      (net 49 "Net-(U3-AVCC)") (pintype "passive"))
     (pad "2" smd roundrect (at 0.775 0) (size 0.9 0.95) (layers "F.Cu" "F.Paste" "F.Mask") (roundrect_rratio 0.25)
       (net 2 "GND") (pintype "passive"))
@@
       (net 2 "GND") (pinfunction "CS") (pintype "input"))
     (pad "2" thru_hole circle locked (at 2.54 -29.26 90) (size 1.8 1.8) (drill 1) (layers "*.Cu" "*.Mask")
-      (net 90 "Net-(#FLG08-pwr)") (pinfunction "RESET") (pintype "input"))
+      (net 90 "Net-(Q10-D)") (pinfunction "RESET") (pintype "input"))
     (pad "3" thru_hole circle locked (at 2.54 -26.72 90) (size 1.8 1.8) (drill 1) (layers "*.Cu" "*.Mask")
       (net 68 "TFT_DC") (pinfunction "DC") (pintype "input"))
@@
       (net 2 "GND") (pinfunction "GND") (pintype "power_in"))
     (pad "11" thru_hole circle locked (at 2.54 -6.4 90) (size 1.8 1.8) (drill 1) (layers "*.Cu" "*.Mask")
-      (net 90 "Net-(#FLG08-pwr)") (pinfunction "VCC") (pintype "power_in"))
+      (net 90 "Net-(Q10-D)") (pinfunction "VCC") (pintype "power_in"))
   )
   (footprint "Resistor_SMD:R_1206_3216Metric" (layer "F.Cu")
@@
       (net 48 "SCK") (pinfunction "PB5") (pintype "bidirectional"))
     (pad "18" smd rect (at 4.25 2) (size 1.6 0.55) (layers "F.Cu" "F.Paste" "F.Mask")
-      (net 49 "Net-(#FLG04-pwr)") (pinfunction "AVCC") (pintype "power_in"))
+      (net 49 "Net-(U3-AVCC)") (pinfunction "AVCC") (pintype "power_in"))
     (pad "19" smd rect (at 4.25 1.2) (size 1.6 0.55) (layers "F.Cu" "F.Paste" "F.Mask")
       (net 97 "unconnected-(U3-ADC6-Pad19)") (pinfunction "ADC6") (pintype "input+no_connect"))
@@
       (net 1 "VCC") (pinfunction "S") (pintype "passive"))
     (pad "3" smd roundrect (at 0.9375 0 180) (size 1.475 0.6) (layers "F.Cu" "F.Paste" "F.Mask") (roundrect_rratio 0.25)
-      (net 90 "Net-(#FLG08-pwr)") (pinfunction "D") (pintype "passive"))
+      (net 90 "Net-(Q10-D)") (pinfunction "D") (pintype "passive"))
     (model "${KICAD6_3DMODEL_DIR}/Package_TO_SOT_SMD.3dshapes/SOT-23.wrl"
       (offset (xyz 0 0 0))
@@
         (effects (font (size 1 1) (thickness 0.15)))
     )
-    (fp_text value "200 pF***" (at 0 1.43 180) (layer "F.Fab") hide
+    (fp_text value "330 pF***" (at 0 1.43 180) (layer "F.Fab") hide
         (effects (font (size 1 1) (thickness 0.15)))
     )
@@
         (effects (font (size 1 1) (thickness 0.15)))
     )
-    (fp_text value "0" (at 0 1.82) (layer "F.Fab") hide
+    (fp_text value "27" (at 0 1.82) (layer "F.Fab") hide
         (effects (font (size 1 1) (thickness 0.15)))
     )
@@
       (stroke (width 0.1) (type solid)) (layer "F.Fab"))
     (pad "1" smd roundrect (at -1.4 0 90) (size 1.25 2.65) (layers "F.Cu" "F.Paste" "F.Mask") (roundrect_rratio 0.2)
-      (net 49 "Net-(#FLG04-pwr)") (pinfunction "1") (pintype "passive"))
+      (net 49 "Net-(U3-AVCC)") (pinfunction "1") (pintype "passive"))
     (pad "2" smd roundrect (at 1.4 0 90) (size 1.25 2.65) (layers "F.Cu" "F.Paste" "F.Mask") (roundrect_rratio 0.2)
       (net 1 "VCC") (pinfunction "2") (pintype "passive"))
@@
     (fp_line (start 8.5 8.75) (end -8.5 8.75)
       (stroke (width 0.12) (type solid)) (layer "F.SilkS"))
-    (fp_arc (start -6.658468 2.010332) (mid -4.996431 0.397649) (end -3.334234 2.010166)
+    (fp_arc (start -6.658468 2.010332) (mid -4.996431 0.397648) (end -3.334234 2.010166)
       (stroke (width 0.12) (type solid)) (layer "F.SilkS"))
-    (fp_arc (start -3.336431 -2.36235) (mid -4.998468 -0.749667) (end -6.660665 -2.362184)
+    (fp_arc (start -3.336431 -2.36235) (mid -4.998468 -0.749666) (end -6.660665 -2.362184)
       (stroke (width 0.12) (type solid)) (layer "F.SilkS"))
-    (fp_arc (start -3.334234 2.010166) (mid -1.672197 0.397482) (end -0.01 2.01)
+    (fp_arc (start -3.334234 2.010166) (mid -1.672197 0.397481) (end -0.01 2.01)
       (stroke (width 0.12) (type solid)) (layer "F.SilkS"))
-    (fp_arc (start -0.012197 -2.362516) (mid -1.674234 -0.749833) (end -3.336431 -2.36235)
+    (fp_arc (start -0.012197 -2.362516) (mid -1.674234 -0.749832) (end -3.336431 -2.36235)
       (stroke (width 0.12) (type solid)) (layer "F.SilkS"))
-    (fp_arc (start -0.01 2.01) (mid 1.652037 0.397316) (end 3.314234 2.009834)
+    (fp_arc (start -0.01 2.01) (mid 1.652037 0.397315) (end 3.314234 2.009834)
       (stroke (width 0.12) (type solid)) (layer "F.SilkS"))
-    (fp_arc (start 3.312037 -2.362682) (mid 1.65 -0.749999) (end -0.012197 -2.362516)
+    (fp_arc (start 3.312037 -2.362682) (mid 1.65 -0.749998) (end -0.012197 -2.362516)
       (stroke (width 0.12) (type solid)) (layer "F.SilkS"))
-    (fp_arc (start 3.314234 2.009834) (mid 4.976271 0.39715) (end 6.638468 2.009668)
+    (fp_arc (start 3.314234 2.009834) (mid 4.976271 0.397149) (end 6.638468 2.009668)
       (stroke (width 0.12) (type solid)) (layer "F.SilkS"))
-    (fp_arc (start 6.636271 -2.362848) (mid 4.974234 -0.750166) (end 3.312037 -2.362682)
+    (fp_arc (start 6.636271 -2.362848) (mid 4.974234 -0.750165) (end 3.312037 -2.362682)
       (stroke (width 0.12) (type solid)) (layer "F.SilkS"))
     (pad "1" thru_hole circle (at -6.5 -7 270) (size 1.8 1.8) (drill 1) (layers "*.Cu" "*.Mask")
@@
         (effects (font (size 1 1) (thickness 0.15)))
     )
-    (fp_text value "VSET [?]" (at 0 1.65) (layer "F.Fab") hide
+    (fp_text value "510K" (at 0 1.65) (layer "F.Fab") hide
         (effects (font (size 1 1) (thickness 0.15)))
     )
@@
       (net 1 "VCC") (pintype "passive"))
     (pad "2" smd roundrect (at 0.9125 0) (size 1.025 1.4) (layers "B.Cu" "B.Paste" "B.Mask") (roundrect_rratio 0.243902)
-      (net 17 "Net-(#FLG03-pwr)") (pintype "passive"))
+      (net 17 "Net-(U1-EN)") (pintype "passive"))
     (model "${KICAD6_3DMODEL_DIR}/Resistor_SMD.3dshapes/R_0805_2012Metric.wrl"
       (offset (xyz 0 0 0))
@@
       (net 2 "GND") (pintype "passive"))
     (pad "2" smd roundrect (at 0.775 0 180) (size 0.9 0.95) (layers "B.Cu" "B.Paste" "B.Mask") (roundrect_rratio 0.25)
-      (net 17 "Net-(#FLG03-pwr)") (pintype "passive"))
+      (net 17 "Net-(U1-EN)") (pintype "passive"))
     (model "${KICAD6_3DMODEL_DIR}/Capacitor_SMD.3dshapes/C_0603_1608Metric.wrl"
       (offset (xyz 0 0 0))
@@
       (net 77 "MCU_I2C_SCL") (pinfunction "SCL2") (pintype "bidirectional"))
     (pad "7" smd roundrect (at 2.1125 0.325 180) (size 1.625 0.4) (layers "B.Cu" "B.Paste" "B.Mask") (roundrect_rratio 0.25)
-      (net 17 "Net-(#FLG03-pwr)") (pinfunction "VREF2") (pintype "power_in"))
+      (net 17 "Net-(U1-EN)") (pinfunction "VREF2") (pintype "power_in"))
     (pad "8" smd roundrect (at 2.1125 0.975 180) (size 1.625 0.4) (layers "B.Cu" "B.Paste" "B.Mask") (roundrect_rratio 0.25)
-      (net 17 "Net-(#FLG03-pwr)") (pinfunction "EN") (pintype "input"))
+      (net 17 "Net-(U1-EN)") (pinfunction "EN") (pintype "input"))
     (model "${KICAD6_3DMODEL_DIR}/Package_SO.3dshapes/MSOP-8_3x3mm_P0.65mm.wrl"
       (offset (xyz 0 0 0))
@@
         (effects (font (size 1 1) (thickness 0.15)) (justify mirror))
     )
-    (fp_text value "400K" (at 0 -1.65) (layer "B.Fab") hide
+    (fp_text value "400K ****" (at 0 -1.65) (layer "B.Fab") hide
         (effects (font (size 1 1) (thickness 0.15)) (justify mirror))
     )
@@
     (property "Sheetfile" "xray.kicad_sch")
     (property "Sheetname" "")
+    (property "ki_description" "Unpolarized capacitor")
+    (property "ki_keywords" "cap capacitor")
     (attr smd)
     (fp_text reference "C33" (at -0.04 2.26 180) (layer "B.SilkS")
