File: schematics/xray/xray.kicad_sch (KiCad schematic)
At the start: 122 parts, among them J1 USB_B_Micro, J2 USB_A, J3 USB_C_Receptacle_USB2.0, J4 USBASP, M1 VibroMotor, 3V, 8x2.7mm, Q1 IRF7832PbF, Q10 IRLML5203, Q11 IRLML0030, Q12 IRLML0030, Q13 IRLML0030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

Commit message: UV power stabilized
Parts:
- R1: value 10 -> 68 **
Other:
- note added: "NOTE* These capacitors used to adjust output voltage NOTE** This resistor can be used to adjust output voltage Use 10...100 ohm to reduce or increase it"
- note removed: "NOTE* These capacitors used to adjust output voltage"
Changed lines of the file:
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@@
     (effects (font (size 1.27 1.27) (thickness 0.254) bold) (justify left bottom))
   )
-  (text "NOTE*\nThese capacitors used to adjust output voltage"
-    (at 95.25 344.17 0)
+  (text "NOTE*\nThese capacitors used to adjust output voltage\n\nNOTE**\nThis resistor can be used to adjust output voltage\nUse 10...100 ohm to reduce or increase it"
+    (at 95.25 351.79 0)
     (effects (font (size 1.27 1.27)) (justify left bottom))
   )
@@
   (symbol (lib_id "Device:R") (at 43.18 313.69 90) (unit 1)
     (in_bom yes) (on_board yes) (dnp no) (fields_autoplaced)
-    (property "Reference" "R1" (at 43.18 307.34 90)
+    (property "Reference" "R1" (at 43.18 308.61 90)
       (effects (font (size 1.27 1.27)))
     )
-    (property "Value" "10" (at 43.18 309.88 90)
+    (property "Value" "68 **" (at 43.18 311.15 90)
       (effects (font (size 1.27 1.27)))
     )
