File: schematics/xray/xray.kicad_sch (KiCad schematic)
At the start: 122 parts, among them J1 USB_B_Micro, J2 USB_A, J3 USB_C_Receptacle_USB2.0, J4 USBASP, M1 VibroMotor, 3V, 8x2.7mm, Q1 IRF7832PbF, Q10 IRLML5203, Q11 IRLML0030, Q12 IRLML0030, Q13 IRLML0030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

Commit message: Start working under EXT STB
Parts:
- C38: value 100 nF -> 2 uF
Changed lines of the file:
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@@
   (symbol (lib_id "Device:C") (at 467.36 238.76 180) (unit 1)
     (in_bom yes) (on_board yes) (dnp no)
-    (property "Reference" "C38" (at 457.2 237.49 0)
+    (property "Reference" "C38" (at 459.74 237.49 0)
       (effects (font (size 1.27 1.27)) (justify right))
     )
-    (property "Value" "100 nF" (at 457.2 240.03 0)
+    (property "Value" "2 uF" (at 459.74 240.03 0)
       (effects (font (size 1.27 1.27)) (justify right))
     )
