File: schematics/xray-v2/xray-v2.kicad_pcb (KiCad board)
At the start: 4 copper layers, 144 x 69 mm, 140 parts, among them J1 USB_B_Micro, J2 USB_B_Micro, J3 USB_A, J4 USB_C_Receptacle_USB2.0, J5 USBASP, M1 VibroMotor, 3V, 8x2.7mm, Q1 IRLML5203, Q10 IRLML0030, Q11 IRLML5203, Q12 IRLML5203, Q13 IRLML0030, Q14 IRLML0030, Q2 IRF7832PbF, Q3 IRF7425PbF, Q4 IRF7425PbF, Q5 IRLML0030, Q6 BC847, Q7 IRLML5203, Q8 IRLML0030, Q9 IRLML0030, SW1 SW_Push, SW2 B3F3150, SW3 EC11W****, T1 Transformer_1P_1S, U1 AMS1117-3.3, U2 CP2102N-Axx-xQFN28, U3 IP5328P, U4 ATmega328P-A, U5 SN74LVC2T45DCUR, U6 SN74LVC2T45DCUR, U7 SN74LVC2T45DCUR, U8 PCA9306, U9 Display_2.2inch_ili9341, Y1 HC-49SM, 8MHz

Commit message: Board v2 ordered. Preparing firmware to work with board-v2
Parts:
- added D1: SMAJ26A, Diode_SMD:D_SMA, F.Cu at (188.1, 120.5)
- added D2: BZV55C3V9, Diode_SMD:D_MiniMELF, F.Cu at (183.0, 123.1)
- moved JP2 0.50 mm to (180.3, 127.1)
- renumbered D1 to D3, D2 to D4, D3 to D5, D4 to D6, D5 to D7, D6 to D8
Connections:
- net RXD_5V renamed RXD_V
- net TXD_5V renamed TXD_V
- JP2 pad 2: FLUSH_VBUS -> CP2102_VREG
Routing:
- net CP2102_VREG: track 3.53 -> 11.7 mm, vias 0 -> 1
- net GND: track 245.4 -> 253.0 mm
- net FLUSH_VBUS: track 16.4 -> 19.5 mm
- net +5V: track 23.2 -> 25.5 mm
Other:
- board text added: "xray v2.1"
- board text removed: "xray v2.0"

Commit message: hardware works, printing box
Parts:
- removed the JP2 at (180.3, 127.1)
- removed JP4: SolderJumper_2_Open, Jumper:SolderJumper-2_P1.3mm_Open_TrianglePad1.0x1.5mm
- added C15: 100 nF, Capacitor_SMD:C_0603_1608Metric, F.Cu at (192.3, 124.6)
- added C18: К73-17, 0.1 uF, 630V, Capacitor_THT:C_Rect_L16.5mm_W7.0mm_P15.00mm_MKT, F.Cu at (164.0, 67.1)
- added D10: BAV21WS, Diode_SMD:D_SOD-323F, F.Cu at (125.8, 127.0)
- added D11: BAV21WS, Diode_SMD:D_SOD-323F, F.Cu at (122.4, 126.4)
- added D12: BAV21WS, Diode_SMD:D_SOD-323F, F.Cu at (119.8, 126.4)
- added D13: BAV21WS, Diode_SMD:D_SOD-323F, F.Cu at (117.2, 126.4)
- added D3: MBR0520, Diode_SMD:D_SOD-123, F.Cu at (183.7, 125.1)
- added D5: US1M, Diode_SMD:D_SMA, B.Cu at (165.7, 75.2)
- added JP3: FL_SPI_EN, Jumper:SolderJumper-2_P1.3mm_Open_TrianglePad1.0x1.5mm, F.Cu at (175.7, 126.9)
- added R25: 10K, Resistor_SMD:R_0805_2012Metric, F.Cu at (179.8, 125.9)
- added R33: 5K, Resistor_SMD:R_0805_2012Metric, B.Cu at (119.8, 129.8)
- added R34: 5K, Resistor_SMD:R_0805_2012Metric, B.Cu at (122.3, 129.8)
- added R35: 5K, Resistor_SMD:R_0805_2012Metric, B.Cu at (124.8, 129.8)
- added TP2: UV_STAB, TestPoint:TestPoint_Pad_1.0x1.0mm, F.Cu at (206.3, 67.9)
- C13: renamed from C12; footprint Capacitor_THT:C_Rect_L16.5mm_W9.0mm_P15.00mm_MKT -> Capacitor_THT:C_Rect_L16.5mm_W7.0mm_P15.00mm_MKT
- C16: renamed from C14; footprint Capacitor_THT:C_Rect_L16.5mm_W9.0mm_P15.00mm_MKT -> Capacitor_THT:C_Rect_L16.5mm_W7.0mm_P15.00mm_MKT
- C20: renamed from C17; footprint Capacitor_THT:C_Rect_L16.5mm_W9.0mm_P15.00mm_MKT -> Capacitor_THT:C_Rect_L16.5mm_W7.0mm_P15.00mm_MKT
- C3, Q1, Q5, R1, R5: moved to B.Cu
- D1: value SMAJ26A -> 15MQ030NPBF
- D2: value BZV55C3V9 -> SP0503BAHT; footprint Diode_SMD:D_MiniMELF -> Package_TO_SOT_SMD:SOT-143
- R10: value 100 -> 510
- TP1: footprint TestPoint:TestPoint_Plated_Hole_D2.0mm -> TestPoint:TestPoint_Loop_D2.54mm_Drill1.5mm_Beaded
- U1: value AMS1117-3.3 -> XC6206P282MR; footprint Package_TO_SOT_SMD:SOT-223-3_TabPin2 -> Package_TO_SOT_SMD:SOT-23-3
- moved D1 48.4 mm to (235.7, 111.6), turned to -90 degrees
- moved D6 13.2 mm to (156.8, 75.1)
- moved R1 13.2 mm to (212.7, 77.9), turned to 180 degrees
- moved D4 13.1 mm to (173.9, 75.2), turned to 0 degrees
- moved TP3 12.5 mm to (194.4, 88.6)
- moved H6 11.5 mm to (204.5, 88.0)
- moved C3 9.79 mm to (212.8, 70.9), turned to 0 degrees
- moved Q1 8.71 mm to (212.6, 74.8), turned to 90 degrees
- moved D2 7.54 mm to (190.1, 120.5), turned to 0 degrees
- moved R5 7.53 mm to (193.4, 90.2), turned to 0 degrees
- moved Q5 7.48 mm to (193.4, 86.4)
- moved C13 6.91 mm to (171.8, 82.1)
- moved C5 6.28 mm to (202.3, 72.4)
- moved C6 6.28 mm to (198.3, 68.4)
- moved C7 6.28 mm to (193.3, 75.4)
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- renumbered C13 to C12, C15 to C14, C16 to C17, C18 to C19, C19 to C21, C20 to C22, C21 to C23, C22 to C24, C23 to C25, C24 to C26, C25 to C27, C26 to C28, C28 to C29, C29 to C30, C30 to C31, C31 to C32, C27 to C33, C32 to C34, C33 to C35, C34 to C36, C35 to C37, C36 to C38, C37 to C39, C38 to C40, C39 to C41, C40 to C42, C41 to C43, C42 to C44, C43 to C45, D8 to D14, D3 to D6, D5 to D7, D6 to D8, D7 to D9, JP3 to JP2, Q11 to Q10, Q10 to Q11, R14 to R11, R11 to R12, R16 to R13, R12 to R14, R13 to R15, R18 to R16, R15 to R17, R17 to R18, R21 to R19, R19 to R20, R20 to R21, R25 to R26, R26 to R27, R27 to R28, R28 to R29, R29 to R30, R30 to R32, R32 to R36, R33 to R37, R34 to R38, R35 to R39, TP2 to TP3, TP3 to TP4, TP4 to TP5, TP5 to TP6
Connections:
- C13 pad 1: Net-(D3-A) -> Net-(D4-K)
- C13 pad 2: Net-(D4-K) -> Net-(T1-SB)
- C16 pad 1: Net-(D3-K) -> GND
- C16 pad 2: GND -> Net-(D5-K)
- C20 pad 2: Net-(D5-K) -> Net-(D7-K)
- D1 pad 1: GND -> USB_M_IN_VBUS
- D2 pad 1: CP2102_VREG -> GND
- D2 pad 2: GND -> FLUSH_VBUS
- D4 pad 2: Net-(D3-K) -> GND
- D6 pad 1: Net-(D3-K) -> Net-(D6-K)
- D6 pad 2: Net-(D3-A) -> Net-(D5-K)
- D7 pad 1: Net-(D5-K) -> Net-(D7-K)
- D7 pad 2: Net-(D4-K) -> Net-(D6-K)
- J5 pad 5: Net-(J5-Pin_5) -> RESET_V
- JP2 pad 2: RESET -> Net-(JP2-B)
- Q10 pad 3: Net-(Q11-D) -> /DISPLAY_VCC
- R10 pad 2: Net-(D5-K) -> Net-(D7-K)
- R12 pad 1: Net-(JP4-B) -> Net-(D7-K)
- T1 pad 4: Net-(D3-A) -> Net-(T1-SB)
- U5 pad 2: RXD -> RESET
- U5 pad 3: MOSI -> RXD
- U5 pad 6: Net-(J5-Pin_1) -> RXD_V
- U5 pad 7: RXD_V -> RESET_V
- U6 pad 2: RESET -> MOSI
- U6 pad 7: Net-(J5-Pin_5) -> Net-(J5-Pin_1)
- U6 pad 8: +5V -> Net-(JP3-A)
- U9 pad 1: Net-(Q11-D) -> /DISPLAY_VCC
- U9 pad 4: Net-(Q11-D) -> Net-(D13-K)
- U9 pad 5: TFT_DC -> Net-(D12-K)
- U9 pad 6: MOSI -> Net-(D11-K)
- U9 pad 7: SCK -> Net-(D10-K)
- U9 pad 8: Net-(Q11-D) -> /DISPLAY_VCC
- U9 pad 9: MISO -> unconnected-(U9-MISO-Pad9)
Routing:
- net FLUSH_VBUS: track 19.5 -> 75.8 mm, vias 1 -> 3
- net Net-(Q11-D): track 44.3 -> 0.00 mm, vias 1 -> 0
- net MISO: track 48.9 -> 6.07 mm
- net Net-(D7-K): track 0.00 -> 39.4 mm
- net /DISPLAY_VCC: track 0.00 -> 36.7 mm, vias 0 -> 2
- net RESET_V: track 0.00 -> 29.3 mm, vias 0 -> 2
- net Net-(D6-K): track 0.00 -> 26.6 mm, vias 0 -> 2
- net USB_M_IN_VBUS: track 27.3 -> 49.6 mm
- net RESET: track 63.1 -> 42.2 mm, vias 4 -> 3
- net Net-(D3-K): track 19.0 -> 0.00 mm
- net Net-(D5-K): track 31.9 -> 14.1 mm
- net Net-(D3-A): track 16.9 -> 0.00 mm
- net Net-(T1-SB): track 0.00 -> 16.1 mm
- net Net-(D4-K): track 27.5 -> 12.0 mm
- net FLUSH_D-: track 7.29 -> 16.7 mm
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Other:
- outline, holes or cut-outs redrawn
- board text added: "xray v2.2.2"
- board text removed: "UV OUT"
- board text removed: "UV PWM"
- board text removed: "xray v2.1"
