File: schematics/xray-v3/xray-v3.kicad_pcb (KiCad board)
At the start: 4 copper layers, 80 x 111 mm, 186 parts, among them J1 TR_SHIELD, J2 USB_C_Receptacle_USB2.0_16P, J3 SBM20_1_+, J4 SBM20_2_+, J5 SBM20_-, J6 SBT9_+, J7 SBT9_-, J8 USB_A, J9 CABEL_SHIELD, Q1 IRLML0060TR, Q2 BC847, Q3 BC847, Q4 IRLML5203, Q5 IRLML5203, Q6 IRLML5203, SW1 SW_SP3T, SW2 START, SW3 RESET, U1 BQ27441DRZR-G1A, U10 SN74LVC1G126DBVR, U11 TPS22965, U12 BQ24090DGQ, U13 TPS22965, U14 INA139, U15 TPS61099DRV, U16 ATtiny1616-M, U17 ATtiny1616-M, U18 RV-3028-C7, U19 LMV331, U2 CP2102N-Axx-xQFN28, U20 SN74LVC2T45DCUR, U21 SN74LVC1T45DCK, U22 XC6206P282MR, U23 Display_2.2inch_ili9341, U3 SN74LVC1G126DBVR, U4 SN74LVC1G126DBVR, U5 SN74LVC1G126DBVR, U6 SN74LVC1T45DCK, U7 SN74LVC1T45DCK, U8 SN74LVC1G126DBVR, U9 SN74LVC1G126DBVR

Commit message: v3.6
Parts:
- removed the C29 at (126.7, 132.1)
- removed D13: BAT54C, Package_TO_SOT_SMD:SOT-23
- removed the D7 at (165.4, 41.1)
- removed the D9 at (158.0, 41.0)
- removed the H3 at (108.0, 66.0)
- removed the JP2 at (160.1, 43.3)
- removed the JP3 at (160.1, 37.6)
- removed JP5: SBT9_EN, Library:SolderedJumper-2P-2mm
- removed the Q5 at (122.4, 109.6)
- removed the R12 at (156.8, 35.7)
- removed the R16 at (151.4, 35.1)
- removed the R40 at (126.6, 130.1)
- removed the R60 at (113.2, 42.4)
- removed TP22: 2.8V, TestPoint:TestPoint_Pad_1.0x1.0mm
- removed the TP7 at (103.5, 117.2)
- removed the U15 at (109.7, 122.4)
- removed the U23 at (105.0, 34.3)
- added C26: 2.2 uF, Capacitor_SMD:C_0603_1608Metric, F.Cu at (116.2, 88.8)
- added C28: 22 uF, Capacitor_SMD:C_1210_3225Metric, B.Cu at (133.9, 117.4)
- added C36: 100 nF, Capacitor_SMD:C_0603_1608Metric, B.Cu at (110.0, 124.0)
- added C37: 47 nF, Capacitor_SMD:C_0603_1608Metric, B.Cu at (107.2, 123.8)
- added C38: 5 nF, Capacitor_SMD:C_0603_1608Metric, F.Cu at (109.8, 116.6)
- added C40: 33 pF, Capacitor_SMD:C_0603_1608Metric, F.Cu at (107.0, 115.8)
- added C41: 100 uF, Capacitor_Tantalum_SMD:CP_EIA-6032-28_Kemet-C_HandSolder, F.Cu at (116.9, 122.6)
- added C42: 22 uF, Capacitor_SMD:C_1210_3225Metric, F.Cu at (113.1, 122.2)
- added C43: 2.2 uF, Capacitor_SMD:C_0603_1608Metric, F.Cu at (126.3, 74.4)
- added C44: 22 uF, Capacitor_SMD:C_1210_3225Metric, F.Cu at (109.7, 122.2)
- added C46: 22 uF, Capacitor_SMD:C_1210_3225Metric, F.Cu at (106.1, 122.2)
- added C47: 100 nF, Capacitor_SMD:C_0603_1608Metric, F.Cu at (127.0, 126.8)
- added C48: 100 nF, Capacitor_SMD:C_0603_1608Metric, F.Cu at (126.6, 120.2)
- added C49: 100 nF, Capacitor_SMD:C_0603_1608Metric, F.Cu at (131.2, 129.2)
- added C51: 100 nF, Capacitor_SMD:C_0603_1608Metric, F.Cu at (133.6, 125.9)
- added C52: 100 nF, Capacitor_SMD:C_0603_1608Metric, B.Cu at (117.4, 50.2)
- added C53: 100 nF, Capacitor_SMD:C_0603_1608Metric, B.Cu at (112.8, 44.4)
- added C55: 100 nF, Capacitor_SMD:C_0603_1608Metric, B.Cu at (119.2, 50.2)
- added C56: 100 nF, Capacitor_SMD:C_0603_1608Metric, F.Cu at (115.2, 43.4)
- added C57: 1 uF, Capacitor_SMD:C_0603_1608Metric, F.Cu at (103.3, 45.6)
- added C61: 47 uF, Capacitor_Tantalum_SMD:CP_EIA-3528-21_Kemet-B_HandSolder, B.Cu at (148.0, 102.2)
- added D10: SP0503BAHT, Package_TO_SOT_SMD:SOT-143, B.Cu at (110.8, 135.0)
- added J10: DSPI, Connector_JST:JST_XH_B4B-XH-A_1x04_P2.50mm_Vertical, F.Cu at (125.6, 41.0)
- added J11: DP/DC, Connector_JST:JST_XH_B2B-XH-A_1x02_P2.50mm_Vertical, F.Cu at (119.4, 35.9)
- added Q6: IRLML5203, Package_TO_SOT_SMD:SOT-23, F.Cu at (125.2, 108.8)
- added Q7: IRLML5203, Package_TO_SOT_SMD:SOT-23, F.Cu at (146.8, 112.2)
- added R33: 100K, Resistor_SMD:R_0805_2012Metric_Pad1.20x1.40mm_HandSolder, F.Cu at (133.8, 122.0)
- added R38: 10K, Resistor_SMD:R_0805_2012Metric_Pad1.20x1.40mm_HandSolder, B.Cu at (110.4, 114.8)
- added R42: 51K, Resistor_SMD:R_0805_2012Metric_Pad1.20x1.40mm_HandSolder, F.Cu at (114.8, 116.8)
- added R45: 17.5K, Resistor_SMD:R_0805_2012Metric_Pad1.20x1.40mm_HandSolder, F.Cu at (107.0, 117.6)
- added R46: 2K, Resistor_SMD:R_0805_2012Metric_Pad1.20x1.40mm_HandSolder, F.Cu at (103.2, 122.4)
- added R48: 0R025, Resistor_SMD:R_2512_6332Metric, F.Cu at (121.8, 122.8)
- added R49: 10K, Resistor_SMD:R_0805_2012Metric_Pad1.20x1.40mm_HandSolder, F.Cu at (126.8, 125.0)
- added R50: 10K, Resistor_SMD:R_0805_2012Metric_Pad1.20x1.40mm_HandSolder, F.Cu at (128.6, 131.4)
- added R58: 10K, Resistor_SMD:R_0805_2012Metric_Pad1.20x1.40mm_HandSolder, F.Cu at (130.8, 124.9)
- added R59: 500, Resistor_SMD:R_0805_2012Metric_Pad1.20x1.40mm_HandSolder, F.Cu at (130.8, 127.2)
- added R66: 10K, Resistor_SMD:R_0805_2012Metric_Pad1.20x1.40mm_HandSolder, F.Cu at (121.8, 108.8)
- added R67: 0 *, Resistor_SMD:R_0805_2012Metric_Pad1.20x1.40mm_HandSolder, F.Cu at (124.4, 46.4)
- added R68: 0 *, Resistor_SMD:R_0805_2012Metric_Pad1.20x1.40mm_HandSolder, F.Cu at (121.2, 43.8)
- added R69: 0 *, Resistor_SMD:R_0805_2012Metric_Pad1.20x1.40mm_HandSolder, F.Cu at (114.2, 37.6)
- added R70: 10K, Resistor_SMD:R_0805_2012Metric_Pad1.20x1.40mm_HandSolder, B.Cu at (134.2, 110.4)
- added U17: INA199A3, Package_TO_SOT_SMD:SOT-363_SC-70-6, F.Cu at (126.2, 122.5)
- added U18: LMV331, Package_TO_SOT_SMD:SOT-23-5_HandSoldering, F.Cu at (125.0, 131.4)
- C1: value 10 nF -> 10 pF
- C10: value ? -> 10 nF *
- C12: value ? -> ? *
- C30: value 100 nF -> 10 uF
- C32: value 4.7 uF -> 10 uF; moved to B.Cu
- C34: value 10 uF -> 100 nF; moved to B.Cu
- C35: value 47 uF -> 2.2 uF; footprint Capacitor_Tantalum_SMD:CP_EIA-3528-21_Kemet-B_HandSolder -> Capacitor_SMD:C_0603_1608Metric; moved to B.Cu
- D1: footprint Diode_SMD:D_MiniMELF_Handsoldering -> Diode_SMD:D_MiniMELF
- D11: renamed from D14; value BAV21 -> BAV21W
- D4, D6: value BAS21S -> BYV26C; footprint Package_TO_SOT_SMD:SOT-23-3 -> Diode_THT:D_5W_P10.16mm_Horizontal
- D5: value BAV21 -> BYV26C; footprint Diode_SMD:D_SOD-123 -> Diode_THT:D_5W_P10.16mm_Horizontal
- D8: value BAS21S -> BAT54C; footprint Package_TO_SOT_SMD:SOT-23-3 -> Package_TO_SOT_SMD:SOT-23; moved to F.Cu
- D9: renamed from D12; value BAV21 -> BAV21W
- J9: value CABEL_SHIELD -> DP/VCC; footprint Connector_JST:JST_XH_B2B-XH-A_1x02_P2.50mm_Vertical -> Connector_JST:JST_XH_B3B-XH-A_1x03_P2.50mm_Vertical
- JP3: renamed from JP6; moved to F.Cu
- L1: value 2.2 uH -> 1 uH; footprint Inductor_SMD:L_Changjiang_FXL0530 -> Inductor_SMD:L_Bourns_SRP1050WA; moved to B.Cu
- R14: renamed from R13; value 300K -> 1M
- R23: renamed from R25; value 1K -> 1K5
- R39: value 0.25 / 4W -> 150K; footprint Library:R_2725 -> Resistor_SMD:R_0805_2012Metric_Pad1.20x1.40mm_HandSolder; moved to B.Cu
- R4: value 10K -> 2K
- R43: value 40K -> 16K
- R44: value 10K -> 100K
- SW1: value SW_SP3T -> SW_SP3T_SH
- SW2: footprint Button_Switch_THT:SW_Tactile_SKHH_Angled -> Library:SW_Tactile_SKHH_Angled_SH
- TP3: footprint TestPoint:TestPoint_2Pads_Pitch2.54mm_Drill0.8mm -> TestPoint:TestPoint_2Pads_Pitch5.08mm_Drill1.3mm; moved to B.Cu
- U14: value INA139 -> TPS61088; footprint Package_TO_SOT_SMD:SOT-23-5 -> Library:VQFN_20; moved to B.Cu
- moved D8 87.6 mm to (133.8, 134.2), turned to 90 degrees
- moved R14 27.5 mm to (178.8, 46.4), turned to 90 degrees
- moved J9 19.5 mm to (108.6, 34.4), turned to 180 degrees
- moved U14 19.0 mm to (105.4, 118.8), turned to -90 degrees
- moved C32 17.0 mm to (126.6, 117.1), turned to 90 degrees
- moved C30 16.7 mm to (133.9, 120.1), turned to 0 degrees
- moved R44 15.7 mm to (102.2, 115.6)
- moved R65 13.2 mm to (108.6, 38.8), turned to 90 degrees
- moved R39 12.9 mm to (110.4, 116.8)
- moved D5 9.92 mm to (166.0, 50.1), turned to 90 degrees
- moved C35 9.46 mm to (101.2, 114.8), turned to -90 degrees
- moved C34 9.36 mm to (111.1, 120.2), turned to 90 degrees
- moved D4 9.09 mm to (170.4, 39.9), turned to -90 degrees
- moved D6 9.08 mm to (161.8, 39.9), turned to -90 degrees
- moved R43 9.07 mm to (111.7, 117.3), turned to 90 degrees
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- renumbered C26 to C27, C27 to C29, C28 to C31, C31 to C33, C33 to C39, C36 to C45, C37 to C50, C38 to C54, C39 to C58, C40 to C59, C41 to C60, D11 to D12, D10 to D7, H4 to H3, H5 to H4, H6 to H5, JP4 to JP2, Q6 to Q5, R14 to R12, R15 to R13, R17 to R15, R18 to R16, R21 to R19, R22 to R20, R30 to R28, R31 to R29, R32 to R30, R33 to R31, R34 to R32, R38 to R37, R41 to R40, R42 to R41, R46 to R47, R47 to R51, R48 to R52, R49 to R53, R45 to R54, R50 to R55, R51 to R56, R52 to R57, R53 to R60, R54 to R61, R58 to R62, R56 to R63, R57 to R64, R59 to R65, R55 to R71, TP12 to TP10, TP13 to TP11, TP15 to TP12, TP14 to TP13, TP16 to TP14, TP17 to TP15, TP9 to TP16, TP18 to TP17, TP19 to TP18, TP20 to TP19, TP21 to TP20, TP8 to TP7, TP10 to TP8, TP11 to TP9, U16 to U15, U17 to U16, U18 to U19, U19 to U20, U20 to U21, U21 to U22, U22 to U23
Connections:
- net /ATTINY_WAKEUP renamed /ATTINY_WAKEUP#
- net Net-(J8-D+) renamed /USBA_D+
- net Net-(J8-D-) renamed /USBA_D-
- C15 pad 2: Net-(D5-K) -> Net-(D4-K)
- C16 pad 2: Net-(D6-A) -> Net-(D5-K)
- C17 pad 1: Net-(D5-K) -> Net-(D4-K)
- C21 pad 1: VCC -> VCOM
- C22 pad 1: VCC -> VCOM
- C29 pad 1: Net-(JP4-B) -> /USB_VIN_IN
- C30 pad 1: Net-(U14-+) -> Net-(U13-ON)
- C32 pad 1: Net-(U14--) -> /USB_VIN
- C34 pad 1: Net-(J8-VBUS) -> Net-(U14-BOOT)
- C34 pad 2: GNDD -> Net-(C34-Pad2)
- C35 pad 1: Net-(J8-VBUS) -> Net-(U14-VCC)
- C39 pad 1: VCC -> VCOM
- C45 pad 1: VCC -> VCOM
- C54 pad 1: VCC -> VCOM
- C7 pad 1: VCC -> VCOM
- C8 pad 1: VCC -> VCOM
- D4 pad 1: Net-(D4-A) -> Net-(D4-K)
- D4 pad 2: Net-(D4-K) -> Net-(D4-A)
- D6 pad 1: Net-(D6-A) -> /HV
- D6 pad 2: Net-(D6-K) -> Net-(D5-K)
- D8 pad 1: Net-(D6-A) -> /USB_OUT_LOCK
- D8 pad 2: Net-(D8-K) -> Net-(D8-Pad2)
- D8 pad 3: unconnected-(D8-common-Pad3) -> Net-(U13-ON)
- J3 pad 1: Net-(J3-Pin_1) -> /HV
- J4 pad 1: Net-(J4-Pin_1) -> /HV
- J6 pad 1: Net-(J6-Pin_1) -> /HV
- J8 pad 1: Net-(J8-VBUS) -> /USBA_VBUS
- J9 pad 1: GND -> /DP_LED
- J9 pad 2: GND -> /DP_VCC
- JP2 pad 2: Net-(JP4-B) -> /USB_VIN_IN
- JP3 pad 1: /DISPLAY_VCC -> /DISPLAY_2.8V
- JP3 pad 2: Net-(JP6-C) -> /DP_VCC
- JP3 pad 3: /DISPLAY_2.8V -> /DISPLAY_VCC
- L1 pad 1: Net-(U14--) -> /USB_VIN
- L1 pad 2: Net-(U15-SW) -> Net-(C34-Pad2)
- Q5 pad 2: VCC -> VCOM
- R14 pad 1: Net-(R12-Pad2) -> GNDPWR
- R14 pad 2: Net-(R13-Pad2) -> Net-(R14-Pad2)
- R32 pad 2: VCC -> VCOM
- R39 pad 1: Net-(U14-+) -> Net-(C34-Pad2)
- R39 pad 2: Net-(U14--) -> Net-(U14-FSW)
- R41 pad 2: VCC -> VCOM
- R43 pad 1: Net-(J8-VBUS) -> Net-(U14-FB)
- R43 pad 2: Net-(U15-FB) -> GNDD
- R44 pad 1: Net-(U15-FB) -> Net-(U14-ILIM)
- R52 pad 1: VCC -> VCOM
- R53 pad 1: VCC -> VCOM
- R62 pad 2: VCC -> VCOM
- R63 pad 1: VCC -> VCOM
- R65 pad 2: Net-(U23-LED) -> /DP_LED
- SW2 pad 1: Net-(JP4-B) -> Net-(D8-Pad2)
- SW2 pad 2: Net-(U13-ON) -> /USB_VIN_IN
- SW3 pad 1: /WAKEUP_BUTTON -> GND
- SW3 pad 2: GND -> /WAKEUP_BUTTON
- TP3 pad 1: Net-(R16-Pad2) -> /HV
- TP3 pad 2: GNDPWR -> Net-(R14-Pad2)
- TR1 pad 2: (no net) -> unconnected-(TR1-NC-Pad2)
- TR1 pad 3: (no net) -> unconnected-(TR1-NC-Pad3)
- U10 pad 5: VCC -> VCOM
- U13 pad 1: Net-(JP4-B) -> /USB_VIN_IN
- U13 pad 2: Net-(JP4-B) -> /USB_VIN_IN
- U13 pad 4: Net-(JP4-B) -> /USB_VIN_IN
- U13 pad 7: Net-(U14-+) -> /USB_VIN
- U13 pad 8: Net-(U14-+) -> /USB_VIN
- U14 pad 1: Net-(U13-ON) -> Net-(U14-VCC)
- U14 pad 2: GNDD -> Net-(U14-EN)
- U14 pad 3: Net-(U14-+) -> Net-(U14-FSW)
- U14 pad 4: Net-(U14--) -> Net-(C34-Pad2)
- U14 pad 5: Net-(U14-+) -> Net-(C34-Pad2)
- U15 pad 4: VCC -> VCOM
- U16 pad 4: VCC -> VCOM
- U19 pad 6: VCC -> VCOM
- U19 pad 7: VCC -> VCOM
- U3 pad 5: VCC -> VCOM
- U4 pad 5: VCC -> VCOM
- U9 pad 5: VCC -> VCOM
Routing:
- net VCOM: track 0.00 -> 195.6 mm, vias 0 -> 5
- net VCC: track 354.7 -> 182.0 mm, vias 6 -> 2
- net GND: track 265.7 -> 165.4 mm, vias 33 -> 37
- net /USB_+5V: track 0.00 -> 72.1 mm, vias 0 -> 1
- net /USB_VIN_IN: track 0.00 -> 41.7 mm, vias 0 -> 4
- net GNDD: track 54.9 -> 95.7 mm, vias 4 -> 6
- net Net-(JP4-B): track 40.0 -> 0.00 mm, vias 1 -> 0
- net Net-(R14-Pad2): track 0.00 -> 38.1 mm
- net GNDPWR: track 162.6 -> 124.6 mm
- net Net-(D9-K): track 54.8 -> 18.9 mm, vias 2 -> 0
- net /USB_VIN: track 0.00 -> 34.5 mm
- net /USBA_VBUS: track 0.00 -> 31.0 mm
- net Net-(U14--): track 29.7 -> 0.00 mm
- net Net-(U14-+): track 21.7 -> 0.00 mm, vias 2 -> 0
- net Net-(J8-VBUS): track 21.6 -> 0.00 mm
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- added copper zone on B.Cu, net /USB_VIN
- added copper zone on B.Cu, net /USB_VIN_IN
Other:
- board text added: "1 UART"
- board text added: "2 UPDI UV"
- board text added: "3 UPDI UI"
- board text added: "xray-v3.6"
- board text removed: "xray-v3.5"
