File: schematics/xray-v3/xray-v3.kicad_pcb (KiCad board)
At the start: 4 copper layers, 80 x 111 mm, 212 parts, among them J1 TR_SHIELD, J10 DSPI, J11 DP/DC, J2 USB_C_Receptacle_USB2.0_16P, J3 SBM20_1_+, J4 SBM20_2_+, J5 SBM20_-, J6 SBT9_+, J7 SBT9_-, J8 USB_A, J9 DP/VCC, Q1 IRLML0060TR, Q2 BC847, Q3 BC847, Q4 IRLML5203, Q5 IRLML5203, Q6 IRLML5203, Q7 IRLML5203, SW1 SW_SP3T_SH, SW2 START, SW3 RESET, U1 BQ27441DRZR-G1A, U10 SN74LVC1G126DBVR, U11 TPS22965, U12 BQ24090DGQ, U13 TPS22965, U14 TPS61088, U15 ATtiny1616-M, U16 ATtiny1616-M, U17 INA199A3, U18 LMV331, U19 RV-3028-C7, U2 CP2102N-Axx-xQFN28, U20 LMV331, U21 SN74LVC2T45DCUR, U22 SN74LVC1T45DCK, U23 XC6206P282MR, U3 SN74LVC1G126DBVR, U4 SN74LVC1G126DBVR, U5 SN74LVC1G126DBVR, U6 SN74LVC1T45DCK, U7 SN74LVC1T45DCK, U8 SN74LVC1G126DBVR, U9 SN74LVC1G126DBVR

Commit message: schematics v3.6.1
Parts:
- added R72: 510K, Resistor_SMD:R_0805_2012Metric_Pad1.20x1.40mm_HandSolder, F.Cu at (102.0, 88.3)
- R42: value 51K -> 22K
- R43: value 16K -> 6K8
- R58: value 10K -> 15K
- R59: value 500 -> 680
Connections:
- C50 pad 2: /WAKEUP_BUTTON -> Net-(Q4-G)
- Q4 pad 1: /WAKEUP_BUTTON -> Net-(Q4-G)
- R51 pad 1: /WAKEUP_BUTTON -> Net-(Q4-G)
- SW3 pad 2: /WAKEUP_BUTTON -> Net-(Q4-G)
Routing:
- net /WAKEUP_BUTTON: track 92.6 -> 42.0 mm
- net Net-(Q4-G): track 0.00 -> 48.6 mm
Other:
- board text added: "xray-v3.6.1"
- board text removed: "xray-v3.6"

Commit message: writing fw
Parts:
- added C62: 10 nF, Capacitor_SMD:C_0603_1608Metric, B.Cu at (158.8, 83.6)
- added C63: 10 nF, Capacitor_SMD:C_0603_1608Metric, B.Cu at (153.2, 83.8)
- added C64: CBB21, 220 nF, 630V, Capacitor_THT:C_Rect_L13.0mm_W6.5mm_P7.50mm_P10.00mm, F.Cu at (155.8, 50.0)
- C15, C16, C17: value CBB21, 10 nF, 630V -> CBB21, 47 nF, 630V
- J3, J4, J6: moved to B.Cu
- R32, R41: value 47K -> 1K5
- moved J3 0.39 mm to (151.8, 37.6), turned to 180 degrees
- moved J4 0.39 mm to (151.8, 43.6), turned to 180 degrees
- moved J6 0.39 mm to (151.8, 49.3), turned to 180 degrees
Routing:
- net GNDPWR: track 124.6 -> 150.7 mm, vias 1 -> 0
- net GND: track 165.4 -> 140.6 mm
- net /HV: track 63.2 -> 56.7 mm
- net /SBM20_SGN_MK: track 14.8 -> 16.5 mm
- net /SBT9_SGM_MK: track 14.8 -> 16.1 mm

Commit message: removed unused line
Parts:
- removed TP1: BS_WKUP, TestPoint:TestPoint_Loop_D2.50mm_Drill1.0mm
Connections:
- R8 pad 1: /BATSTATE_WAKEUP -> Net-(U1-BIN)
- U1 pad 10: /BATSTATE_WAKEUP -> Net-(U1-BIN)
- U15 pad 10: /BATSTATE_WAKEUP -> unconnected-(U15-PB4-Pad10)
Routing:
- net /BATSTATE_WAKEUP: track 115.0 -> 0.00 mm, vias 2 -> 0
- net Net-(U1-BIN): track 0.00 -> 8.76 mm
- net /HV: track 56.7 -> 55.4 mm
