File: schematics/xray-v3/xray-v3.kicad_sch (KiCad schematic)
At the start: 200 parts, among them J1 TR_SHIELD, J2 USB_C_Receptacle_USB2.0_16P, J3 SBM20_1_+, J4 SBM20_2_+, J5 SBM20_-, J6 SBT9_+, J7 SBT9_-, J8 USB_A, J9 CABEL_SHIELD, Q1 IRLML0060TR, Q2 BC847, Q3 BC847, Q4 IRLML5203, Q5 IRLML5203, Q6 IRLML5203, SW1 SW_SP3T, SW2 START, SW3 RESET, U1 BQ27441DRZR-G1A, U10 SN74LVC1G126DBVR, U11 TPS22965, U12 BQ24090DGQ, U13 TPS22965, U14 INA139, U15 TPS61099DRV, U16 ATtiny1616-M, U17 ATtiny1616-M, U18 RV-3028-C7, U19 LMV331, U2 CP2102N-Axx-xQFN28, U20 SN74LVC2T45DCUR, U21 SN74LVC1T45DCK, U22 XC6206P282MR, U23 Display_2.2inch_ili9341, U3 SN74LVC1G126DBVR, U4 SN74LVC1G126DBVR, U5 SN74LVC1G126DBVR, U6 SN74LVC1T45DCK, U7 SN74LVC1T45DCK, U8 SN74LVC1G126DBVR, U9 SN74LVC1G126DBVR

Commit message: v3.6
Parts:
- removed C29: 10 nF, Capacitor_SMD:C_0603_1608Metric, symbol Device:C
- removed C35: 47 uF, Capacitor_Tantalum_SMD:CP_EIA-3528-21_Kemet-B_HandSolder, symbol Device:C_Polarized
- removed D13: BAT54C, Package_TO_SOT_SMD:SOT-23, symbol Diode:BAT54C
- removed D4, D6, D8: BAS21S, Package_TO_SOT_SMD:SOT-23-3, symbol Device:D_Dual_Series_AKC
- removed D5, D7, D9: BAV21W, Diode_SMD:D_SOD-123, symbol Diode:BAV21
- removed H3: MountingHole, MountingHole:MountingHole_2.2mm_M2, symbol Mechanical:MountingHole
- removed J9: CABEL_SHIELD, Connector_JST:JST_XH_B2B-XH-A_1x02_P2.50mm_Vertical, symbol Connector:Conn_01x02_Socket
- removed JP2: SBM20_2_EN, Library:SolderedJumper-2P-2mm, symbol Jumper:SolderJumper_2_Open
- removed JP3: SBM20_1_EN, Library:SolderedJumper-2P-2mm, symbol Jumper:SolderJumper_2_Open
- removed JP5: SBT9_EN, Library:SolderedJumper-2P-2mm, symbol Jumper:SolderJumper_2_Open
- removed Q5: IRLML5203, Package_TO_SOT_SMD:SOT-23, symbol Transistor_FET:IRLML5203
- removed R12, R16: 300K, Resistor_SMD:R_0805_2012Metric_Pad1.20x1.40mm_HandSolder, symbol Device:R
- removed R40: 200K, Resistor_SMD:R_0805_2012Metric_Pad1.20x1.40mm_HandSolder, symbol Device:R
- removed R60: 1M, Resistor_SMD:R_0805_2012Metric_Pad1.20x1.40mm_HandSolder, symbol Device:R
- removed SW1: SW_SP3T, Library:SK13D07VG4, symbol Switch:SW_SP3T
- removed SW2: START, Button_Switch_THT:SW_Tactile_SKHH_Angled, symbol Switch:SW_Push
- removed TP22: 2.8V, TestPoint:TestPoint_Pad_1.0x1.0mm, symbol Connector:TestPoint
- removed TP7: USB_PWR, TestPoint:TestPoint_Loop_D2.50mm_Drill1.0mm, symbol Connector:TestPoint
- removed U14: INA139, Package_TO_SOT_SMD:SOT-23-5, symbol Amplifier_Current:INA139
- removed U15: TPS61099DRV, Package_SON:WSON-6-1EP_2x2mm_P0.65mm_EP1x1.6mm, symbol Regulator_Switching:TPS61099DRV
- added C26, C35, C43: 2.2 uF, Capacitor_SMD:C_0603_1608Metric, symbol Device:C
- added C28, C42, C44, C46: 22 uF, Capacitor_SMD:C_1210_3225Metric, symbol Device:C
- added C36, C47, C48, C49, C51, C52, C53, C55, C56: 100 nF, Capacitor_SMD:C_0603_1608Metric, symbol Device:C
- added C37: 47 nF, Capacitor_SMD:C_0603_1608Metric, symbol Device:C
- added C38: 5 nF, Capacitor_SMD:C_0603_1608Metric, symbol Device:C
- added C40: 33 pF, Capacitor_SMD:C_0603_1608Metric, symbol Device:C
- added C41: 100 uF, Capacitor_Tantalum_SMD:CP_EIA-6032-28_Kemet-C_HandSolder, symbol Device:C_Polarized
- added C57: 1 uF, Capacitor_SMD:C_0603_1608Metric, symbol Device:C
- added C61: 47 uF, Capacitor_Tantalum_SMD:CP_EIA-3528-21_Kemet-B_HandSolder, symbol Device:C_Polarized
- added D10: SP0503BAHT, Package_TO_SOT_SMD:SOT-143, symbol Power_Protection:SP0503BAHT
- added D4, D5, D6: BYV26C, Diode_THT:D_5W_P10.16mm_Horizontal, symbol Device:D
- added D8: BAT54C, Package_TO_SOT_SMD:SOT-23, symbol Diode:BAT54C
- added J10: DSPI, Connector_JST:JST_XH_B4B-XH-A_1x04_P2.50mm_Vertical, symbol Connector:Conn_01x04_Socket
- added J11: DP/DC, Connector_JST:JST_XH_B2B-XH-A_1x02_P2.50mm_Vertical, symbol Connector:Conn_01x02_Socket
- added J12: Conn_01x06_Pin, symbol Connector:Conn_01x06_Pin
- added J9: DP/VCC, Connector_JST:JST_XH_B3B-XH-A_1x03_P2.50mm_Vertical, symbol Connector:Conn_01x03_Socket
- added Q6, Q7: IRLML5203, Package_TO_SOT_SMD:SOT-23, symbol Transistor_FET:IRLML5203
- added R33: 100K, Resistor_SMD:R_0805_2012Metric_Pad1.20x1.40mm_HandSolder, symbol Device:R
- added R38, R49, R50, R58, R66, R70: 10K, Resistor_SMD:R_0805_2012Metric_Pad1.20x1.40mm_HandSolder, symbol Device:R
- added R42: 51K, Resistor_SMD:R_0805_2012Metric_Pad1.20x1.40mm_HandSolder, symbol Device:R
- added R45: 17.5K, Resistor_SMD:R_0805_2012Metric_Pad1.20x1.40mm_HandSolder, symbol Device:R
- added R46: 2K, Resistor_SMD:R_0805_2012Metric_Pad1.20x1.40mm_HandSolder, symbol Device:R
- added R48: 0R025, Resistor_SMD:R_2512_6332Metric, symbol Device:R
- added R59: 500, Resistor_SMD:R_0805_2012Metric_Pad1.20x1.40mm_HandSolder, symbol Device:R
- added R67, R68, R69: 0 *, Resistor_SMD:R_0805_2012Metric_Pad1.20x1.40mm_HandSolder, symbol Device:R
- added SW1: SW_SP3T_SH, Library:SK13D07VG4, symbol My_Library:SW_SP3T_SH
- added SW2: START, Library:SW_Tactile_SKHH_Angled_SH, symbol Switch:CK_KMS2xxG
- added U14: TPS61088, Library:VQFN_20, symbol My_Library:TPS61088
- added U17: INA199A3, Package_TO_SOT_SMD:SOT-363_SC-70-6, symbol Amplifier_Current:INA199xxDCK
- added U18: LMV331, Package_TO_SOT_SMD:SOT-23-5_HandSoldering, symbol Comparator:LMV331
- C10: value ? -> 10 nF *
- C12: value ? -> ? *
- C30: value 100 nF -> 10 uF
- C32: value 4.7 uF -> 10 uF
- C34: value 10 uF -> 100 nF
- D1: footprint Diode_SMD:D_MiniMELF_Handsoldering -> Diode_SMD:D_MiniMELF
- L1: value 2.2 uH -> 1 uH; footprint Inductor_SMD:L_Changjiang_FXL0530 -> Inductor_SMD:L_Bourns_SRP1050WA
- R14: renamed from R13; value 300K -> 1M
- R39: value 0.25 / 4W -> 150K; footprint Library:R_2725 -> Resistor_SMD:R_0805_2012Metric_Pad1.20x1.40mm_HandSolder
- R4: value 4K7 -> 2K
- R43: value 40K -> 16K
- R44: value 10K -> 100K
- TP3: footprint TestPoint:TestPoint_2Pads_Pitch2.54mm_Drill0.8mm -> TestPoint:TestPoint_2Pads_Pitch5.08mm_Drill1.3mm
- renumbered C26 to C27, C27 to C29, C28 to C31, C31 to C33, C33 to C39, C36 to C45, C37 to C50, C38 to C54, C39 to C58, C40 to C59, C41 to C60, D14 to D11, D11 to D12, D10 to D7, D12 to D9, H4 to H3, H5 to H4, H6 to H5, JP4 to JP2, JP6 to JP3, Q6 to Q5, R14 to R12, R15 to R13, R17 to R15, R18 to R16, R19 to R17, R20 to R18, R21 to R19, R22 to R20, R23 to R21, R24 to R22, R25 to R23, R26 to R24, R27 to R25, R28 to R26, R29 to R27, R30 to R28, R31 to R29, R32 to R30, R33 to R31, R34 to R32, R35 to R34, R36 to R35, R37 to R36, R38 to R37, R41 to R40, R42 to R41, R46 to R47, R47 to R51, R48 to R52, R49 to R53, R45 to R54, R50 to R55, R51 to R56, R52 to R57, R53 to R60, R54 to R61, R58 to R62, R56 to R63, R57 to R64, R59 to R65, R55 to R71, TP12 to TP10, TP13 to TP11, TP15 to TP12, TP14 to TP13, TP16 to TP14, TP17 to TP15, TP9 to TP16, TP18 to TP17, TP19 to TP18, TP20 to TP19, TP21 to TP20, TP8 to TP7, TP10 to TP8, TP11 to TP9, U16 to U15, U17 to U16, U18 to U19, U19 to U20, U20 to U21, U21 to U22, U22 to U23, U23 to U24
Connections:
- net DISPLAY_2.8V: now also JP3.1 (A), C55.1, C56.1; no longer JP3.3 (B), U24.4 (RESET#)
- net DISPLAY_VCC: now also JP3.3 (B), C52.1, C53.1, C57.1; no longer JP3.1 (A)
- net GND: now also SW3.1, C26.2, C43.2, C52.2, C53.2, C55.2, C56.2, C57.2, C61.2, J10.1 (Pin_1), J10.3 (Pin_3), J11.2 (Pin_2), J9.3 (Pin_3), R70.1, SW1.SH; no longer SW3.2, U24.2 (GND), U24.3 (CS)
- net GNDD: now also R43.2, C28.2, C35.2, C36.2, C37.2, C38.2, C40.2, C41.2, C42.2, C44.2, C46.2, C47.2, C48.2, C49.2, C51.2, D10.1 (A), R33.1, R46.1, R59.2, SW2.SH (B), U14.20 (AGND), U14.EXP (PGND), U17.1 (REF), U17.2 (GND), U18.2 (V-); no longer C34.2
- net GNDPWR: now also R14.1; no longer TP3.2
- net HV: now also J3.1 (Pin_1), J4.1 (Pin_1), J6.1 (Pin_1), R17.1, R18.1, R34.1, TP3.1, D6.1 (K)
- net UART_EN: now also SW1.1
- net UPDI1_EN: now also SW1.2
- net UPDI2_EN: now also SW1.4
- net VCC: now also Q7.2 (S); no longer C21.1, C22.1, C39.1, C45.1, C54.1, C7.1, C8.1, Q5.2 (S), R32.2, R41.2, R52.1, R53.1, R62.2, R63.1, U10.5 (VCC), U15.4 (VCC), U16.4 (VCC), U19.6 (VBACKUP), U19.7 (VDD), U3.5 (VCC), U4.5 (VCC), U9.5 (VCC)
- net VCCQ: now also C26.1, SW1.3
- net WAKEUP_BUTTON: now also SW3.2; no longer SW3.1
- net at U13.3 (ON): now also C30.1, D8.3, R33.2
- net USB_VIN: now reaches U13.7 (VOUT), U13.8 (VOUT)
- net USB_VIN: now also C32.1, L1.1, C36.1, R38.1, U14.9 (VIN); no longer C30.1, R39.1
- net at R44.1: now also U14.19 (ILIM); no longer R43.2
- net at C15.2, C17.1: now also D4.1 (K), D5.2 (A)
- net at U21.6 (B2): now also R68.2; no longer U24.6 (MOSI)
- net at U21.7 (B1): now also R67.2; no longer U24.7 (SCK)
- net at D9.1 (K), TP16.1, U20.4: now also Q6.1 (G), R66.1
- net USB_VIN_IN: now reaches C29.1, JP2.2 (B), U13.1 (VIN), U13.2 (VIN), U13.4 (VBIAS)
- net USB_VIN_IN: now also C28.1, SW2.2
- net at C16.1, TR1.5: now also D4.2 (A)
- net at C16.2: now also D5.1 (K), D6.2 (A)
- net at D11.1 (K), Q4.3 (D), R60.2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: now also Q6.2 (S), R66.2
- net at U24.8 (LED): now also J12.1 (Pin_1); no longer R65.2
- net at R14.2: now also TP3.2
- net at L1.2: now also C34.2, R39.1, U14.4 (SW), U14.5 (SW), U14.6 (SW), U14.7 (SW)
- net at U24.1 (VCC): now also U24.4 (RESET#), J12.2 (Pin_2); no longer JP3.2 (C)
- net at U24.5 (DC): now also J12.5 (Pin_5); no longer U22.4 (B)
- net USBA_D-: now reaches J8.2 (D-), R54.2
- net USBA_D-: now also D10.3 (K)
- net USBA_D+: now reaches J8.3 (D+), R54.1
- net USBA_D+: now also D10.4 (K)
- net at D12.2 (A): now also Q6.3 (D), Q7.1 (G), R70.2
- new net: C40.1, R45.1, U14.18 (COMP)
- new net: D8.2, SW2.1
- new net: R38.2, U14.2 (EN)
- new net: C38.1, R45.2
- new net: R42.2, R43.1, U14.17 (FB)
- new net: C34.1, U14.8 (BOOT)
- new net: C35.1, U14.1 (VCC)
- new net: R49.1, U17.6
- new net: C47.1, R49.2, U18.1 (+)
- new net: J12.3 (Pin_3), U24.7 (SCK)
- new net: J12.4 (Pin_4), U24.6 (MOSI)
- new net: J12.6 (Pin_6), U24.2 (GND), U24.3 (CS)
- new net: C37.1, U14.10 (SS)
- new net: R39.2, U14.3 (FSW)
- new net: R58.2, R59.1, U18.3 (-)
- new net: R69.1, U22.4 (B)
- new net DP_DC: J11.1 (Pin_1), R69.2
- new net DP_LED: J9.1 (Pin_1), R65.2
- new net DP_MOSI: J10.4 (Pin_4), R68.1
- new net DP_SCK: J10.2 (Pin_2), R67.1
- new net DP_VCC: J9.2 (Pin_2), JP3.2 (C)
- new net USBA_VBUS: D10.2 (K), J8.1 (VBUS), R48.2, U17.5 (-)
- new net USB_+5V: C41.1, C42.1, C44.1, C46.1, C48.1, C49.1, C51.1, R42.1, R46.2, R48.1, R50.1, R58.1, U14.14 (VOUT), U14.15 (VOUT), U14.16 (VOUT), U17.3 (V+), U17.4 (+), U18.5 (V+)
- new net USB_OUT_LOCK: D8.1, R50.2, U18.4
- new net VCOM: C21.1, C22.1, C39.1, C43.1, C45.1, C54.1, C61.1, C7.1, C8.1, Q5.2 (S), Q7.3 (D), R32.2, R41.2, R52.1, R53.1, R62.2, R63.1, U10.5 (VCC), U15.4 (VCC), U16.4 (VCC), U19.6 (VBACKUP), U19.7 (VDD), U3.5 (VCC), U4.5 (VCC), U9.5 (VCC)
- no-connect marks 35 -> 33
Other:
- moved on the sheet: C15, C16, C17, C29, C50, C58, C59, C60, D11, D12, D9, H3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
