File: schematics/xray-v3/xray-v3.kicad_sch (KiCad schematic)
At the start: 228 parts, among them J1 TR_SHIELD, J10 DSPI, J11 DP/DC, J12 Conn_01x06_Pin, J2 USB_C_Receptacle_USB2.0_16P, J3 SBM20_1_+, J4 SBM20_2_+, J5 SBM20_-, J6 SBT9_+, J7 SBT9_-, J8 USB_A, J9 DP/VCC, Q1 IRLML0060TR, Q2 BC847, Q3 BC847, Q4 IRLML5203, Q5 IRLML5203, Q6 IRLML5203, Q7 IRLML5203, SW1 SW_SP3T_SH, SW2 START, SW3 RESET, U1 BQ27441DRZR-G1A, U10 SN74LVC1G126DBVR, U11 TPS22965, U12 BQ24090DGQ, U13 TPS22965, U14 TPS61088, U15 ATtiny1616-M, U16 ATtiny1616-M, U17 INA199A3, U18 LMV331, U19 RV-3028-C7, U2 CP2102N-Axx-xQFN28, U20 LMV331, U21 SN74LVC2T45DCUR, U22 SN74LVC1T45DCK, U23 XC6206P282MR, U24 Display_2.2inch_ili9341, U3 SN74LVC1G126DBVR, U4 SN74LVC1G126DBVR, U5 SN74LVC1G126DBVR, U6 SN74LVC1T45DCK, U7 SN74LVC1T45DCK, U8 SN74LVC1G126DBVR, U9 SN74LVC1G126DBVR

Commit message: schematics v3.6.1
Parts:
- added R72: 510K, Resistor_SMD:R_0805_2012Metric_Pad1.20x1.40mm_HandSolder, symbol Device:R
- C1: now not fitted
- R42: value 51K -> 22K
- R43: value 16K -> 6K8
- R58: value 10K -> 15K
- R59: value 500 -> 680
Connections:
- net WAKEUP_BUTTON: now also R72.2; no longer C50.2, Q4.1 (G), R51.1, SW3.2
- new net: C50.2, Q4.1 (G), R51.1, R72.1, SW3.2
Changed lines of the file:
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@@
 	(wire
 		(pts
+			(xy 575.31 168.91) (xy 579.12 168.91)
+		)
+		(stroke
+			(width 0)
+			(type default)
+		)
+	)
+	(wire
+		(pts
 			(xy 566.42 45.72) (xy 576.58 45.72)
 		)
@@
 	(wire
 		(pts
-			(xy 586.74 168.91) (xy 596.9 168.91)
-		)
-		(stroke
-			(width 0)
-			(type default)
-		)
-	)
-	(wire
-		(pts
 			(xy 542.29 49.53) (xy 542.29 45.72)
 		)
@@
 	(wire
 		(pts
+			(xy 586.74 168.91) (xy 596.9 168.91)
+		)
+		(stroke
+			(width 0)
+			(type default)
+		)
+	)
+	(wire
+		(pts
 			(xy 762 29.21) (xy 762 33.02)
 		)
@@
 	)
 	(label "WAKEUP_BUTTON"
-		(at 586.74 168.91 180)
+		(at 575.31 168.91 180)
 		(effects
 			(font
@@
 			)
 		)
-		(property "Value" "51K"
+		(property "Value" "22K"
 			(at 476.25 52.0699 0)
 			(show_name no)
@@
 	)
 	(symbol
+		(lib_id "Device:R")
+		(at 582.93 168.91 270)
+		(unit 1)
+		(body_style 1)
+		(exclude_from_sim no)
+		(in_bom yes)
+		(on_board yes)
+		(in_pos_files yes)
+		(dnp no)
+		(property "Reference" "R72"
+			(at 581.025 172.085 90)
+			(show_name no)
+			(do_not_autoplace no)
+			(effects
+				(font
+					(size 1.27 1.27)
+				)
+				(justify left)
+			)
+		)
+		(property "Value" "510K"
+			(at 581.025 174.625 90)
+			(show_name no)
+			(do_not_autoplace no)
+			(effects
+				(font
+					(size 1.27 1.27)
+				)
+				(justify left)
+			)
+		)
+		(property "Footprint" "Resistor_SMD:R_0805_2012Metric_Pad1.20x1.40mm_HandSolder"
+			(at 582.93 167.132 90)
+			(hide yes)
+			(show_name no)
+			(do_not_autoplace no)
+			(effects
+				(font
+					(size 1.27 1.27)
+				)
+			)
+		)
+		(property "Datasheet" ""
+			(at 582.93 168.91 0)
+			(hide yes)
+			(show_name no)
+			(do_not_autoplace no)
+			(effects
+				(font
+					(size 1.27 1.27)
+				)
+			)
+		)
+		(property "Description" "Resistor"
+			(at 582.93 168.91 0)
+			(hide yes)
+			(show_name no)
+			(do_not_autoplace no)
+			(effects
+				(font
+					(size 1.27 1.27)
+				)
+			)
+		)
+		(pin "1"
+		)
+		(pin "2"
+		)
+		(instances
+			(project "xray-v3"
+				(path "/dd8f4371-6f2d-42cc-9067-2496b53ad747"
+					(reference "R72")
+					(unit 1)
+				)
+			)
+		)
+	)
+	(symbol
 		(lib_id "power:GND")
 		(at 673.1 439.42 0)
@@
 		(dnp no)
 		(property "Reference" "Q4"
-			(at 631.19 142.24 0)
+			(at 614.172 137.668 0)
 			(show_name no)
 			(do_not_autoplace no)
@@
 		)
 		(property "Value" "IRLML5203"
-			(at 631.19 144.78 0)
+			(at 614.172 140.208 0)
 			(show_name no)
 			(do_not_autoplace no)
@@
 			)
 		)
-		(property "Value" "16K"
+		(property "Value" "6K8"
 			(at 485.902 53.34 90)
 			(show_name no)
@@
 			)
 		)
-		(property "Value" "500"
+		(property "Value" "680"
 			(at 628.65 85.0899 0)
 			(show_name no)
@@
 		(on_board yes)
 		(in_pos_files yes)
-		(dnp no)
+		(dnp yes)
 		(property "Reference" "C1"
 			(at 52.324 547.878 0)
@@
 			)
 		)
-		(property "Value" "10K"
+		(property "Value" "15K"
 			(at 628.65 74.9299 0)
 			(show_name no)

Commit message: writing fw
Parts:
- added C62, C63: 10 nF, Capacitor_SMD:C_0603_1608Metric, symbol Device:C
- added C64: CBB21, 220 nF, 630V, Capacitor_THT:C_Rect_L13.0mm_W6.5mm_P7.50mm_P10.00mm, symbol Device:C
- C15, C16, C17: value CBB21, 10 nF, 630V -> CBB21, 47 nF, 630V
- R32, R41: value 47K -> 1K5
Connections:
- net GND: now also C62.2, C63.2
- net GNDPWR: now also C64.1
- net HV: now also C64.2
- net SBM20_SGN_MK: now also C62.1
- net SBT9_SGM_MK: now also C63.1

Commit message: removed unused line
Parts:
- removed TP1: BS_WKUP, TestPoint:TestPoint_Loop_D2.50mm_Drill1.0mm, symbol Connector:TestPoint
Connections:
- net BATSTATE_WAKEUP: no longer names the net of R8.1, U1.10 (BIN)
- net BATSTATE_WAKEUP: no longer U15.10 (PB4)
- no-connect marks 33 -> 34
Other:
- moved on the sheet: R8
Changed lines of the file:
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@@
 	)
 	(junction
-		(at 74.93 60.96)
-		(diameter 0)
-		(color 0 0 0 0)
-	)
-	(junction
 		(at 59.69 542.29)
 		(diameter 0)
@@
 	)
 	(no_connect
+		(at 544.83 434.34)
+	)
+	(no_connect
 		(at 121.92 247.65)
 	)
@@
 	(wire
 		(pts
-			(xy 74.93 44.45) (xy 74.93 60.96)
+			(xy 74.93 44.45) (xy 74.93 49.53)
 		)
 		(stroke
@@
 	(wire
 		(pts
-			(xy 74.93 60.96) (xy 77.47 60.96)
-		)
-		(stroke
-			(width 0)
-			(type default)
-		)
-	)
-	(wire
-		(pts
 			(xy 60.96 58.42) (xy 60.96 62.23)
 		)
@@
 	(wire
 		(pts
-			(xy 74.93 69.85) (xy 74.93 71.12)
+			(xy 74.93 57.15) (xy 74.93 58.42)
 		)
 		(stroke
@@
 	(wire
 		(pts
-			(xy 544.83 434.34) (xy 548.64 434.34)
-		)
-		(stroke
-			(width 0)
-			(type default)
-		)
-	)
-	(wire
-		(pts
 			(xy 300.99 133.35) (xy 300.99 137.16)
 		)
@@
 	(wire
 		(pts
-			(xy 66.04 86.36) (xy 66.04 90.17)
-		)
-		(stroke
-			(width 0)
-			(type default)
-		)
-	)
-	(wire
-		(pts
 			(xy 459.74 519.43) (xy 459.74 521.97)
 		)
@@
 	(wire
 		(pts
-			(xy 74.93 60.96) (xy 74.93 62.23)
-		)
-		(stroke
-			(width 0)
-			(type default)
-		)
-	)
-	(wire
-		(pts
 			(xy 740.41 434.34) (xy 745.49 434.34)
 		)
@@
 		)
 	)
-	(label "BATSTATE_WAKEUP"
-		(at 548.64 434.34 0)
-		(effects
-			(font
-				(size 1.27 1.27)
-			)
-			(justify left bottom)
-		)
-	)
 	(label "USB1_VBUS"
 		(at 231.14 140.97 180)
@@
 		)
 	)
-	(label "BATSTATE_WAKEUP"
-		(at 66.04 90.17 180)
-		(effects
-			(font
-				(size 1.27 1.27)
-			)
-			(justify right bottom)
-		)
-	)
 	(label "USB1_TX_VCC"
 		(at 130.81 440.69 180)
@@
 		)
 	)
-	(label "BATSTATE_WAKEUP"
-		(at 77.47 60.96 0)
-		(effects
-			(font
-				(size 1.27 1.27)
-			)
-			(justify left bottom)
-		)
-	)
 	(label "SBT9_SGM_MK"
 		(at 476.25 521.97 0)
@@
 	)
 	(symbol
-		(lib_id "Connector:TestPoint")
-		(at 66.04 86.36 0)
-		(unit 1)
-		(body_style 1)
-		(exclude_from_sim no)
-		(in_bom yes)
-		(on_board yes)
-		(in_pos_files yes)
-		(dnp no)
-		(fields_autoplaced yes)
-		(property "Reference" "TP1"
-			(at 68.58 81.7879 0)
-			(show_name no)
-			(do_not_autoplace no)
-			(effects
-				(font
-					(size 1.27 1.27)
-				)
-				(justify left)
-			)
-		)
-		(property "Value" "BS_WKUP"
-			(at 68.58 84.3279 0)
-			(show_name no)
-			(do_not_autoplace no)
-			(effects
-				(font
-					(size 1.27 1.27)
-				)
-				(justify left)
-			)
-		)
-		(property "Footprint" "TestPoint:TestPoint_Loop_D2.50mm_Drill1.0mm"
-			(at 71.12 86.36 0)
-			(hide yes)
-			(show_name no)
-			(do_not_autoplace no)
-			(effects
-				(font
-					(size 1.27 1.27)
-				)
-			)
-		)
-		(property "Datasheet" ""
-			(at 71.12 86.36 0)
-			(hide yes)
-			(show_name no)
-			(do_not_autoplace no)
-			(effects
-				(font
-					(size 1.27 1.27)
-				)
-			)
-		)
-		(property "Description" "test point"
-			(at 66.04 86.36 0)
-			(hide yes)
-			(show_name no)
-			(do_not_autoplace no)
-			(effects
-				(font
-					(size 1.27 1.27)
-				)
-			)
-		)
-		(pin "1"
-		)
-		(instances
-			(project "xray-v3"
-				(path "/dd8f4371-6f2d-42cc-9067-2496b53ad747"
-					(reference "TP1")
-					(unit 1)
-				)
-			)
-		)
-	)
-	(symbol
 		(lib_id "power:GNDD")
 		(at 673.1 64.77 0)
@@
 	(symbol
 		(lib_id "Device:R")
-		(at 74.93 66.04 0)
+		(at 74.93 53.34 0)
 		(unit 1)
 		(body_style 1)
@@
 		(fields_autoplaced yes)
 		(property "Reference" "R8"
-			(at 77.47 64.7699 0)
+			(at 77.47 52.0699 0)
 			(show_name no)
 			(do_not_autoplace no)
@@
 		)
 		(property "Value" "10K"
-			(at 77.47 67.3099 0)
+			(at 77.47 54.6099 0)
 			(show_name no)
 			(do_not_autoplace no)
@@
 		)
 		(property "Footprint" "Resistor_SMD:R_0805_2012Metric_Pad1.20x1.40mm_HandSolder"
-			(at 73.152 66.04 90)
+			(at 73.152 53.34 90)
 			(hide yes)
 			(show_name no)
@@
 		)
 		(property "Datasheet" ""
-			(at 74.93 66.04 0)
+			(at 74.93 53.34 0)
 			(hide yes)
 			(show_name no)
@@
 		)
 		(property "Description" "Resistor"
-			(at 74.93 66.04 0)
+			(at 74.93 53.34 0)
 			(hide yes)
 			(show_name no)
@@
 	(symbol
 		(lib_id "power:GND")
-		(at 74.93 71.12 0)
+		(at 74.93 58.42 0)
 		(unit 1)
 		(body_style 1)
@@
 		(fields_autoplaced yes)
 		(property "Reference" "#PWR017"
-			(at 74.93 77.47 0)
+			(at 74.93 64.77 0)
 			(hide yes)
 			(show_name no)
@@
 		)
 		(property "Value" "GND"
-			(at 74.93 76.2 0)
+			(at 74.93 63.5 0)
 			(show_name no)
 			(do_not_autoplace no)
@@
 		)
 		(property "Footprint" ""
-			(at 74.93 71.12 0)
+			(at 74.93 58.42 0)
 			(hide yes)
 			(show_name no)
@@
 		)
 		(property "Datasheet" ""
-			(at 74.93 71.12 0)
+			(at 74.93 58.42 0)
 			(hide yes)
 			(show_name no)
@@
 		)
 		(property "Description" "Power symbol creates a global label with name \"GND\" , ground"
-			(at 74.93 71.12 0)
+			(at 74.93 58.42 0)
 			(hide yes)
 			(show_name no)
